File: mm_motor.kicad_sch (KiCad schematic)
At the start: 1 part, among them M1 N20_encoder

Commit message: fin tp2
Parts:
- added C7: 10uf, symbol Device:C
- added J2: Conn_01x06_Pin, Connector_PinHeader_2.54mm:PinHeader_1x06_P2.54mm_Vertical, symbol Connector:Conn_01x06_Pin
Connections:
- net C1: now also J2.3 (Pin_3)
- net C2: now also J2.4 (Pin_4)
- net MA: now also J2.1 (Pin_1)
- net MB: now also J2.6 (Pin_6)
- new net +BATT: C7.2, J2.5 (Pin_5)
- new net GND: C7.1, J2.2 (Pin_2)
Changed lines of the file:
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@@
 (kicad_sch (version 20230121) (generator eeschema)
   (paper "A4")
-  (hierarchical_label "C1" (shape output) (at 118.11 91.44 180) (fields_autoplaced)
-    (effects (font (size 1.27 1.27)) (justify right))
-  )
-  (hierarchical_label "C2" (shape output) (at 118.11 93.98 180) (fields_autoplaced)
-    (effects (font (size 1.27 1.27)) (justify right))
-  )
-  (hierarchical_label "MB" (shape passive) (at 118.11 99.06 180) (fields_autoplaced)
-    (effects (font (size 1.27 1.27)) (justify right))
-  )
-  (hierarchical_label "MA" (shape passive) (at 118.11 86.36 180) (fields_autoplaced)
-    (effects (font (size 1.27 1.27)) (justify right))
+  (junction (at 109.22 72.39) (diameter 0) (color 0 0 0 0)
+  )
+  (wire (pts (xy 100.33 93.98) (xy 118.11 93.98))
+    (stroke (width 0) (type default))
+  )
+  (wire (pts (xy 100.33 88.9) (xy 104.14 88.9))
+    (stroke (width 0) (type default))
+  )
+  (wire (pts (xy 109.22 72.39) (xy 116.84 72.39))
+    (stroke (width 0) (type default))
+  )
+  (wire (pts (xy 104.14 88.9) (xy 104.14 107.95))
+    (stroke (width 0) (type default))
+  )
+  (wire (pts (xy 109.22 72.39) (xy 109.22 96.52))
+    (stroke (width 0) (type default))
+  )
+  (wire (pts (xy 100.33 86.36) (xy 118.11 86.36))
+    (stroke (width 0) (type default))
+  )
+  (wire (pts (xy 100.33 91.44) (xy 118.11 91.44))
+    (stroke (width 0) (type default))
+  )
+  (wire (pts (xy 100.33 99.06) (xy 118.11 99.06))
+    (stroke (width 0) (type default))
+  )
+  (wire (pts (xy 109.22 96.52) (xy 100.33 96.52))
+    (stroke (width 0) (type default))
+  )
+  (wire (pts (xy 109.22 68.58) (xy 109.22 72.39))
+    (stroke (width 0) (type default))
+  )
+  (wire (pts (xy 116.84 80.01) (xy 116.84 110.49))
+    (stroke (width 0) (type default))
+  )
+  (hierarchical_label "C1" (shape output) (at 118.11 91.44 0) (fields_autoplaced)
+    (effects (font (size 1.27 1.27)) (justify left))
+  )
+  (hierarchical_label "C2" (shape output) (at 118.11 93.98 0) (fields_autoplaced)
+    (effects (font (size 1.27 1.27)) (justify left))
+  )
+  (hierarchical_label "MB" (shape passive) (at 118.11 99.06 0) (fields_autoplaced)
+    (effects (font (size 1.27 1.27)) (justify left))
+  )
+  (hierarchical_label "MA" (shape passive) (at 118.11 86.36 0) (fields_autoplaced)
+    (effects (font (size 1.27 1.27)) (justify left))
+  )
+  (symbol (lib_id "Connector:Conn_01x06_Pin") (at 95.25 91.44 0) (unit 1)
+    (in_bom yes) (on_board yes) (dnp no) (fields_autoplaced)
+    (property "Reference" "J2" (at 95.885 81.28 0)
+      (effects (font (size 1.27 1.27)))
+    )
+    (property "Value" "Conn_01x06_Pin" (at 95.885 83.82 0)
+      (effects (font (size 1.27 1.27)))
+    )
+    (property "Footprint" "Connector_PinHeader_2.54mm:PinHeader_1x06_P2.54mm_Vertical" (at 95.25 91.44 0)
+      (effects (font (size 1.27 1.27)) hide)
+    )
+    (property "Datasheet" "~" (at 95.25 91.44 0)
+      (effects (font (size 1.27 1.27)) hide)
+    )
+    (pin "6")
+    (pin "1")
+    (pin "4")
+    (pin "3")
+    (pin "5")
+    (pin "2")
+    (instances
+      (project "minimouse"
+        (path "/d8fa4cba-2469-4231-847f-065b6b829f44/7f113667-692a-4f4d-b16f-621d32f3f136"
+          (reference "J2") (unit 1)
+        )
+        (path "/d8fa4cba-2469-4231-847f-065b6b829f44/3975acd0-18ad-47bc-9ce1-d8c4d864aafe"
+          (reference "J3") (unit 1)
+        )
+      )
+    )
   )
   (symbol (lib_id "minimouse:N20_w_encoder") (at 115.57 57.15 0) (unit 1)
@@
         )
       )
+    )
+  )
+  (symbol (lib_id "power:+BATT") (at 109.22 68.58 0) (unit 1)
+    (in_bom yes) (on_board yes) (dnp no) (fields_autoplaced)
+    (property "Reference" "#PWR028" (at 109.22 72.39 0)
+      (effects (font (size 1.27 1.27)) hide)
+    )
+    (property "Value" "+BATT" (at 109.22 63.5 0)
+      (effects (font (size 1.27 1.27)))
+    )
+    (property "Footprint" "" (at 109.22 68.58 0)
+      (effects (font (size 1.27 1.27)) hide)
+    )
+    (property "Datasheet" "" (at 109.22 68.58 0)
+      (effects (font (size 1.27 1.27)) hide)
+    )
+    (pin "1")
+    (instances
+      (project "minimouse"
+        (path "/d8fa4cba-2469-4231-847f-065b6b829f44/7f113667-692a-4f4d-b16f-621d32f3f136"
+          (reference "#PWR028") (unit 1)
+        )
+        (path "/d8fa4cba-2469-4231-847f-065b6b829f44/3975acd0-18ad-47bc-9ce1-d8c4d864aafe"
+          (reference "#PWR029") (unit 1)
+        )
+      )
+    )
+  )
+  (symbol (lib_id "power:GND") (at 116.84 110.49 0) (unit 1)
+    (in_bom yes) (on_board yes) (dnp no) (fields_autoplaced)
+    (property "Reference" "#PWR035" (at 116.84 116.84 0)
+      (effects (font (size 1.27 1.27)) hide)
+    )
+    (property "Value" "GND" (at 116.84 115.57 0)
+      (effects (font (size 1.27 1.27)))
+    )
+    (property "Footprint" "" (at 116.84 110.49 0)
+      (effects (font (size 1.27 1.27)) hide)
+    )
+    (property "Datasheet" "" (at 116.84 110.49 0)
+      (effects (font (size 1.27 1.27)) hide)
+    )
+    (pin "1")
+    (instances
+      (project "minimouse"
+        (path "/d8fa4cba-2469-4231-847f-065b6b829f44/7f113667-692a-4f4d-b16f-621d32f3f136"
+          (reference "#PWR035") (unit 1)
+        )
+        (path "/d8fa4cba-2469-4231-847f-065b6b829f44/3975acd0-18ad-47bc-9ce1-d8c4d864aafe"
+          (reference "#PWR038") (unit 1)
+        )
+      )
+    )
+  )
+  (symbol (lib_id "Device:C") (at 116.84 76.2 180) (unit 1)
+    (in_bom yes) (on_board yes) (dnp no) (fields_autoplaced)
+    (property "Reference" "C7" (at 120.65 74.93 0)
+      (effects (font (size 1.27 1.27)) (justify right))
+    )
+    (property "Value" "10uf" (at 120.65 77.47 0)
+      (effects (font (size 1.27 1.27)) (justify right))
+    )
+    (property "Footprint" "" (at 115.8748 72.39 0)
+      (effects (font (size 1.27 1.27)) hide)
+    )
+    (property "Datasheet" "~" (at 116.84 76.2 0)
+      (effects (font (size 1.27 1.27)) hide)
+    )
+    (pin "2")
+    (pin "1")
+    (instances
+      (project "minimouse"
+        (path "/d8fa4cba-2469-4231-847f-065b6b829f44/d17bb1c7-f68a-465e-9a17-5858ef86fc30"
+          (reference "C7") (unit 1)
+        )
+        (path "/d8fa4cba-2469-4231-847f-065b6b829f44/7f113667-692a-4f4d-b16f-621d32f3f136"
+          (reference "C10") (unit 1)
+        )
+        (path "/d8fa4cba-2469-4231-847f-065b6b829f44/3975acd0-18ad-47bc-9ce1-d8c4d864aafe"
+          (reference "C11") (unit 1)
+        )
+      )
+    )
+  )
+  (symbol (lib_id "power:GND") (at 104.14 107.95 0) (unit 1)
+    (in_bom yes) (on_board yes) (dnp no) (fields_autoplaced)
+    (property "Reference" "#PWR026" (at 104.14 114.3 0)
+      (effects (font (size 1.27 1.27)) hide)
+    )
+    (property "Value" "GND" (at 104.14 113.03 0)
+      (effects (font (size 1.27 1.27)))
+    )
+    (property "Footprint" "" (at 104.14 107.95 0)
+      (effects (font (size 1.27 1.27)) hide)
+    )
+    (property "Datasheet" "" (at 104.14 107.95 0)
+      (effects (font (size 1.27 1.27)) hide)
+    )
+    (pin "1")
+    (instances
+      (project "minimouse"
+        (path "/d8fa4cba-2469-4231-847f-065b6b829f44/7f113667-692a-4f4d-b16f-621d32f3f136"
+          (reference "#PWR026") (unit 1)
+        )
+        (path "/d8fa4cba-2469-4231-847f-065b6b829f44/3975acd0-18ad-47bc-9ce1-d8c4d864aafe"
+          (reference "#PWR027") (unit 1)
+        )
+      )

Commit message: TP3
Parts:
- added R12, R14: 100, Resistor_SMD:R_0603_1608Metric, symbol Device:R
- C10: renamed from C7; value 10uf -> 2.2uf; footprint (none) -> Capacitor_SMD:C_0603_1608Metric
Connections:
- net C1: now also R12.2; no longer J2.3 (Pin_3)
- net C2: now also R14.2; no longer J2.4 (Pin_4)
- new net: J2.3 (Pin_3), R12.1
- new net: J2.4 (Pin_4), R14.1
Other:
- moved on the sheet: C10, M1
Changed lines of the file:
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@@
 (kicad_sch (version 20230121) (generator eeschema)
   (paper "A4")
-  (junction (at 109.22 72.39) (diameter 0) (color 0 0 0 0)
-  )
-  (wire (pts (xy 100.33 93.98) (xy 118.11 93.98))
+  (wire (pts (xy 100.33 91.44) (xy 113.03 91.44))
+    (stroke (width 0) (type default))
+  )
+  (wire (pts (xy 120.65 91.44) (xy 128.27 91.44))
     (stroke (width 0) (type default))
   )
@@
     (stroke (width 0) (type default))
   )
-  (wire (pts (xy 109.22 72.39) (xy 116.84 72.39))
-    (stroke (width 0) (type default))
-  )
   (wire (pts (xy 104.14 88.9) (xy 104.14 107.95))
     (stroke (width 0) (type default))
   )
-  (wire (pts (xy 109.22 72.39) (xy 109.22 96.52))
+  (wire (pts (xy 109.22 68.58) (xy 109.22 96.52))
     (stroke (width 0) (type default))
   )
@@
     (stroke (width 0) (type default))
   )
-  (wire (pts (xy 100.33 91.44) (xy 118.11 91.44))
-    (stroke (width 0) (type default))
-  )
   (wire (pts (xy 100.33 99.06) (xy 118.11 99.06))
     (stroke (width 0) (type default))
@@
     (stroke (width 0) (type default))
   )
-  (wire (pts (xy 109.22 68.58) (xy 109.22 72.39))
-    (stroke (width 0) (type default))
-  )
-  (wire (pts (xy 116.84 80.01) (xy 116.84 110.49))
-    (stroke (width 0) (type default))
-  )
-  (hierarchical_label "C1" (shape output) (at 118.11 91.44 0) (fields_autoplaced)
-    (effects (font (size 1.27 1.27)) (justify left))
-  )
-  (hierarchical_label "C2" (shape output) (at 118.11 93.98 0) (fields_autoplaced)
+  (wire (pts (xy 100.33 93.98) (xy 113.03 93.98))
+    (stroke (width 0) (type default))
+  )
+  (wire (pts (xy 143.51 82.55) (xy 143.51 90.17))
+    (stroke (width 0) (type default))
+  )
+  (wire (pts (xy 120.65 93.98) (xy 128.27 93.98))
+    (stroke (width 0) (type default))
+  )
+  (wire (pts (xy 143.51 97.79) (xy 143.51 105.41))
+    (stroke (width 0) (type default))
+  )
+  (hierarchical_label "C1" (shape output) (at 128.27 91.44 0) (fields_autoplaced)
+    (effects (font (size 1.27 1.27)) (justify left))
+  )
+  (hierarchical_label "C2" (shape output) (at 128.27 93.98 0) (fields_autoplaced)
     (effects (font (size 1.27 1.27)) (justify left))
   )
@@
     )
   )
-  (symbol (lib_id "minimouse:N20_w_encoder") (at 115.57 57.15 0) (unit 1)
-    (in_bom yes) (on_board yes) (dnp no) (fields_autoplaced)
-    (property "Reference" "M1" (at 118.11 55.88 0)
+  (symbol (lib_id "power:+BATT") (at 143.51 82.55 0) (unit 1)
+    (in_bom yes) (on_board yes) (dnp no) (fields_autoplaced)
+    (property "Reference" "#PWR044" (at 143.51 86.36 0)
+      (effects (font (size 1.27 1.27)) hide)
+    )
+    (property "Value" "+BATT" (at 143.51 77.47 0)
+      (effects (font (size 1.27 1.27)))
+    )
+    (property "Footprint" "" (at 143.51 82.55 0)
+      (effects (font (size 1.27 1.27)) hide)
+    )
+    (property "Datasheet" "" (at 143.51 82.55 0)
+      (effects (font (size 1.27 1.27)) hide)
+    )
+    (pin "1")
+    (instances
+      (project "minimouse"
+        (path "/d8fa4cba-2469-4231-847f-065b6b829f44/7f113667-692a-4f4d-b16f-621d32f3f136"
+          (reference "#PWR044") (unit 1)
+        )
+        (path "/d8fa4cba-2469-4231-847f-065b6b829f44/3975acd0-18ad-47bc-9ce1-d8c4d864aafe"
+          (reference "#PWR045") (unit 1)
+        )
+      )
+    )
+  )
+  (symbol (lib_id "minimouse:N20_w_encoder") (at 119.38 74.93 0) (unit 1)
+    (in_bom yes) (on_board yes) (dnp no) (fields_autoplaced)
+    (property "Reference" "M1" (at 121.92 73.66 0)
       (effects (font (size 1.27 1.27)) (justify left))
     )
-    (property "Value" "N20_encoder" (at 118.11 58.42 0)
+    (property "Value" "N20_encoder" (at 121.92 76.2 0)
       (effects (font (size 1.27 1.27)) (justify left))
     )
-    (property "Footprint" "minimouse:N20_with_encoder" (at 118.11 53.34 0)
-      (effects (font (size 1.27 1.27)) hide)
-    )
-    (property "Datasheet" "" (at 115.57 57.15 0)
+    (property "Footprint" "minimouse:N20_with_encoder" (at 121.92 71.12 0)
+      (effects (font (size 1.27 1.27)) hide)
+    )
+    (property "Datasheet" "" (at 119.38 74.93 0)
       (effects (font (size 1.27 1.27)) hide)
     )
@@
     )
   )
-  (symbol (lib_id "power:GND") (at 116.84 110.49 0) (unit 1)
-    (in_bom yes) (on_board yes) (dnp no) (fields_autoplaced)
-    (property "Reference" "#PWR035" (at 116.84 116.84 0)
-      (effects (font (size 1.27 1.27)) hide)
-    )
-    (property "Value" "GND" (at 116.84 115.57 0)
-      (effects (font (size 1.27 1.27)))
-    )
-    (property "Footprint" "" (at 116.84 110.49 0)
-      (effects (font (size 1.27 1.27)) hide)
-    )
-    (property "Datasheet" "" (at 116.84 110.49 0)
+  (symbol (lib_id "Device:R") (at 116.84 93.98 90) (unit 1)
+    (in_bom yes) (on_board yes) (dnp no)
+    (property "Reference" "R14" (at 116.84 96.52 90)
+      (effects (font (size 1.27 1.27)))
+    )
+    (property "Value" "100" (at 121.92 95.25 90)
+      (effects (font (size 1.27 1.27)))
+    )
+    (property "Footprint" "Resistor_SMD:R_0603_1608Metric" (at 116.84 95.758 90)
+      (effects (font (size 1.27 1.27)) hide)
+    )
+    (property "Datasheet" "~" (at 116.84 93.98 0)
+      (effects (font (size 1.27 1.27)) hide)
+    )
+    (pin "2")
+    (pin "1")
+    (instances
+      (project "minimouse"
+        (path "/d8fa4cba-2469-4231-847f-065b6b829f44/7f113667-692a-4f4d-b16f-621d32f3f136"
+          (reference "R14") (unit 1)
+        )
+        (path "/d8fa4cba-2469-4231-847f-065b6b829f44/3975acd0-18ad-47bc-9ce1-d8c4d864aafe"
+          (reference "R15") (unit 1)
+        )
+      )
+    )
+  )
+  (symbol (lib_id "power:GND") (at 143.51 105.41 0) (unit 1)
+    (in_bom yes) (on_board yes) (dnp no) (fields_autoplaced)
+    (property "Reference" "#PWR035" (at 143.51 111.76 0)
+      (effects (font (size 1.27 1.27)) hide)
+    )
+    (property "Value" "GND" (at 143.51 110.49 0)
+      (effects (font (size 1.27 1.27)))
+    )
+    (property "Footprint" "" (at 143.51 105.41 0)
+      (effects (font (size 1.27 1.27)) hide)
+    )
+    (property "Datasheet" "" (at 143.51 105.41 0)
       (effects (font (size 1.27 1.27)) hide)
     )
@@
     )
   )
-  (symbol (lib_id "Device:C") (at 116.84 76.2 180) (unit 1)
-    (in_bom yes) (on_board yes) (dnp no) (fields_autoplaced)
-    (property "Reference" "C7" (at 120.65 74.93 0)
+  (symbol (lib_id "Device:R") (at 116.84 91.44 90) (unit 1)
+    (in_bom yes) (on_board yes) (dnp no)
+    (property "Reference" "R12" (at 116.84 88.9 90)
+      (effects (font (size 1.27 1.27)))
+    )
+    (property "Value" "100" (at 121.92 90.17 90)
+      (effects (font (size 1.27 1.27)))
+    )
+    (property "Footprint" "Resistor_SMD:R_0603_1608Metric" (at 116.84 93.218 90)
+      (effects (font (size 1.27 1.27)) hide)
+    )
+    (property "Datasheet" "~" (at 116.84 91.44 0)
+      (effects (font (size 1.27 1.27)) hide)
+    )
+    (pin "2")
+    (pin "1")
+    (instances
+      (project "minimouse"
+        (path "/d8fa4cba-2469-4231-847f-065b6b829f44/7f113667-692a-4f4d-b16f-621d32f3f136"
+          (reference "R12") (unit 1)
+        )
+        (path "/d8fa4cba-2469-4231-847f-065b6b829f44/3975acd0-18ad-47bc-9ce1-d8c4d864aafe"
+          (reference "R13") (unit 1)
+        )
+      )
+    )
+  )
+  (symbol (lib_id "Device:C") (at 143.51 93.98 180) (unit 1)
+    (in_bom yes) (on_board yes) (dnp no)
+    (property "Reference" "C10" (at 147.32 92.71 0)
       (effects (font (size 1.27 1.27)) (justify right))
     )
-    (property "Value" "10uf" (at 120.65 77.47 0)
+    (property "Value" "2.2uf" (at 147.32 95.25 0)
       (effects (font (size 1.27 1.27)) (justify right))
     )
-    (property "Footprint" "" (at 115.8748 72.39 0)
-      (effects (font (size 1.27 1.27)) hide)
-    )
-    (property "Datasheet" "~" (at 116.84 76.2 0)
-      (effects (font (size 1.27 1.27)) hide)
-    )
-    (pin "2")
-    (pin "1")
-    (instances
-      (project "minimouse"
-        (path "/d8fa4cba-2469-4231-847f-065b6b829f44/d17bb1c7-f68a-465e-9a17-5858ef86fc30"
-          (reference "C7") (unit 1)
-        )
+    (property "Footprint" "Capacitor_SMD:C_0603_1608Metric" (at 142.5448 90.17 0)
+      (effects (font (size 1.27 1.27)) hide)
+    )
+    (property "Datasheet" "~" (at 143.51 93.98 0)
+      (effects (font (size 1.27 1.27)) hide)
+    )
+    (pin "2")
+    (pin "1")
+    (instances
+      (project "minimouse"
         (path "/d8fa4cba-2469-4231-847f-065b6b829f44/7f113667-692a-4f4d-b16f-621d32f3f136"
           (reference "C10") (unit 1)
