File: mm_motor_control.kicad_sch (KiCad schematic)
At the start: 0 parts

Commit message: fin tp2
Parts:
- added C7: 10uf, symbol Device:C
- added CEN: 10nf, symbol Device:C
- added CROFF, CSPOL: 22UF, symbol Device:C
- added CS: 2.2UF, symbol Device:C
- added CSTBY: 1nf, symbol Device:C
- added R50, R51: 2.2k, symbol Device:R
- added R52, R53: 18k, symbol Device:R
- added R54: 47k, symbol Device:R
- added R55: 1k, symbol Device:R
- added R56, R57: 330m, symbol Device:R
- added U2: STSPIN240, Package_DFN_QFN:VQFN-16-1EP_3x3mm_P0.5mm_EP1.8x1.8mm, symbol Driver_Motor:STSPIN240
Connections:
- net EN: now also R53.1
- net FAULT: now also CEN.1, R53.2, U2.13 (EN/FLT)
- net OUT_A1: now also U2.3 (OUTA1)
- net OUT_A2: now also U2.5 (OUTA2)
- net OUT_B1: now also U2.10 (OUTB1)
- net OUT_B2: now also U2.8 (OUTB2)
- net PHASE_A: now also U2.1 (PHA)
- net PHASE_B: now also U2.15 (PHB)
- net PWM_A: now also U2.2 (PWMA)
- net PWM_B: now also U2.16 (PWMB)
- net STBY/RESET: now also CSTBY.1, R52.2, U2.14 (STBY/RESET)
- new net: R50.1, R51.2, U2.11 (REF)
- new net: R57.1, U2.4 (SENSEA)
- new net: R56.1, U2.9 (SENSEB)
- new net: R54.1, R55.1, U2.12 (TOFF)
- new net: CROFF.1, R55.2
- new net +3V3: R52.1
- new net +BATT: C7.2, CS.1, CSPOL.1, R50.2, U2.6 (VS)
- new net GND: C7.1, CEN.2, CROFF.2, CS.2, CSPOL.2, CSTBY.2, R51.1, R54.2, R56.2, R57.2, U2.17 (EPAD), U2.7 (GND)

Commit message: TP3
Parts:
- removed C7: 10uf, symbol Device:C
- removed CSPOL: 22UF, symbol Device:C
- removed CSTBY: 1nf, symbol Device:C
- removed R52: 18k, symbol Device:R
- C75: renamed from CROFF; value 22UF -> 22nF; footprint (none) -> Capacitor_SMD:C_0603_1608Metric
- C80: renamed from CEN; value 10nf -> 1nf; footprint (none) -> Capacitor_SMD:C_0603_1608Metric
- CS1: renamed from CS; footprint (none) -> Capacitor_SMD:C_0603_1608Metric
- R50, R51: value 2.2k -> 10k; footprint (none) -> Resistor_SMD:R_0603_1608Metric
- R53, R54, R55: footprint (none) -> Resistor_SMD:R_0603_1608Metric
- R56, R57: footprint (none) -> Resistor_SMD:R_2512_6332Metric
Connections:
- net GND: now also R57.1; no longer R57.2
- net at U2.4 (SENSEA): now also R57.2; no longer R57.1
Other:
- moved on the sheet: R57
