File: mm_power.kicad_sch (KiCad schematic)
At the start: 1 part, among them J5 Conn_01x02

Commit message: fin tp2
Parts:
- added CIN, COUT: 1uf, symbol Device:C
- added D2: LED, LED_SMD:LED_0603_1608Metric_Pad1.05x0.95mm_HandSolder, symbol Device:LED
- added R10: 120, symbol Device:R
- added U3: LP5907MFX-3.3, Package_TO_SOT_SMD:SOT-23-5, symbol Regulator_Linear:LP5907MFX-3.3
Connections:
- net +BATT: now also CIN.1, U3.1 (IN), U3.3 (EN)
- net GND: now also CIN.2, COUT.2, R10.2, U3.2 (GND)
- new net: D2.1 (K), R10.1
- new net +3V3: COUT.1, D2.2 (A), U3.5 (OUT)

Commit message: TP3
Parts:
- C81: renamed from CIN; value 1uf -> 2.2uf; footprint (none) -> Capacitor_SMD:C_0603_1608Metric
- C82: renamed from COUT; value 1uf -> 2.2uf; footprint (none) -> Capacitor_SMD:C_0603_1608Metric
- D2: footprint LED_SMD:LED_0603_1608Metric_Pad1.05x0.95mm_HandSolder -> LED_SMD:LED_0603_1608Metric
- R10: value 120 -> 330; footprint (none) -> Resistor_SMD:R_0603_1608Metric
Connections:
- net GND: now also D2.1 (K); no longer R10.2
- net +3.3V: now reaches R10.1
- net +3.3V: now also C82.1, U3.5 (OUT); no longer D2.1 (K)
- removed net +3V3: C82.1, D2.2 (A), U3.5 (OUT)
- new net: D2.2 (A), R10.2
