File: minimouse.kicad_pcb (KiCad board)
At the start: 2 copper layers, 90 x 85 mm, 22 parts, among them J1 Conn_ARM_JTAG_SWD_10, J5 Conn_01x02, M1 N20_encoder, M2 N20_encoder, U1 STM32F030C8Tx, U4 HC-SR04

Commit message: TP3
Parts:
- added C10: 2.2uf, Capacitor_SMD:C_0603_1608Metric, F.Cu at (174.8, 100.6)
- added C11: 2.2uf, Capacitor_SMD:C_0603_1608Metric, F.Cu at (125.1, 99.7)
- added C12: 2.2uF, Capacitor_SMD:C_0603_1608Metric, F.Cu at (145.1, 71.8)
- added C75: 22nF, Capacitor_SMD:C_0603_1608Metric, F.Cu at (158.9, 105.6)
- added C8: 2.2uf, Capacitor_SMD:C_0603_1608Metric, F.Cu at (161.0, 75.0)
- added C80: 1nf, Capacitor_SMD:C_0603_1608Metric, F.Cu at (150.8, 102.5)
- added C81: 2.2uf, Capacitor_SMD:C_0603_1608Metric, F.Cu at (126.1, 84.2)
- added C82: 2.2uf, Capacitor_SMD:C_0603_1608Metric, F.Cu at (129.2, 76.9)
- added CS1: 2.2UF, Capacitor_SMD:C_0603_1608Metric, F.Cu at (158.9, 109.4)
- added D2: LED, LED_SMD:LED_0603_1608Metric, F.Cu at (129.2, 82.0)
- added J2: Conn_01x06_Pin, Connector_PinHeader_2.54mm:PinHeader_1x06_P2.54mm_Vertical, F.Cu at (165.2, 97.5)
- added J3: Conn_01x06_Pin, Connector_PinHeader_2.54mm:PinHeader_1x06_P2.54mm_Vertical, F.Cu at (135.4, 96.7)
- added J4: Conn_01x04_Pin, Connector_PinHeader_2.54mm:PinHeader_1x04_P2.54mm_Vertical, F.Cu at (160.2, 72.1)
- added R10: 330, Resistor_SMD:R_0603_1608Metric, F.Cu at (125.2, 76.9)
- added R11: 100, Resistor_SMD:R_0603_1608Metric, F.Cu at (151.3, 71.9)
- added R12: 100, Resistor_SMD:R_0603_1608Metric, F.Cu at (168.2, 100.6)
- added R13: 100, Resistor_SMD:R_0603_1608Metric, F.Cu at (132.5, 99.7)
- added R14: 100, Resistor_SMD:R_0603_1608Metric, F.Cu at (171.7, 100.6)
- added R15: 100, Resistor_SMD:R_0603_1608Metric, F.Cu at (128.7, 99.7)
- added R16: 100, Resistor_SMD:R_0603_1608Metric, F.Cu at (165.0, 75.0)
- added R50: 10k, Resistor_SMD:R_0603_1608Metric, F.Cu at (154.6, 110.2)
- added R51: 10k, Resistor_SMD:R_0603_1608Metric, F.Cu at (154.6, 107.6)
- added R53: 18k, Resistor_SMD:R_0603_1608Metric, F.Cu at (150.8, 105.1)
- added R54: 47k, Resistor_SMD:R_0603_1608Metric, F.Cu at (154.6, 105.1)
- added R55: 1k, Resistor_SMD:R_0603_1608Metric, F.Cu at (154.6, 103.6)
- added R56: 330m, Resistor_SMD:R_2512_6332Metric, F.Cu at (154.7, 114.0)
- added R57: 330m, Resistor_SMD:R_2512_6332Metric, F.Cu at (142.8, 107.6)
- added U2: STSPIN240, Package_DFN_QFN:VQFN-16-1EP_3x3mm_P0.5mm_EP1.8x1.8mm, F.Cu at (150.2, 108.7)
- added U3: LP5907MFX-3.3, Package_TO_SOT_SMD:SOT-23-5, F.Cu at (125.7, 80.6)
- moved C5 10.1 mm to (134.1, 92.0)
- moved BOOT0 3.82 mm to (157.4, 82.0)
- moved R2 2.57 mm to (142.8, 98.0)
- moved J1 2.47 mm to (161.4, 83.2)
- moved R3 2.42 mm to (145.0, 98.0)
- moved R4 2.42 mm to (146.5, 98.0)
- moved R5 2.42 mm to (148.0, 98.0)
- moved C2 1.96 mm to (146.1, 81.1)
- moved C6 1.88 mm to (144.3, 81.1)
- moved R6 1.55 mm to (150.5, 97.9)
- moved R7 1.55 mm to (152.0, 97.9)
- moved C1 1.06 mm to (142.0, 91.2)
- moved C3 0.93 mm to (142.0, 87.6)
- moved R9 0.75 mm to (147.8, 81.1)
- moved R8 0.50 mm to (151.8, 81.1)
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Connections:
- R8 pad 1: /mcu/UART1_TX -> /external_uart/EXT_UART_RX
- U1 pad 43: /mcu/UART1_RX -> /external_uart/EXT_UART_TX

Commit message: tp4
Parts:
- moved R8 16.6 mm to (167.7, 76.4)
- moved R12 12.8 mm to (155.6, 98.7)
- moved R13 12.0 mm to (142.0, 92.3)
- moved R16 11.7 mm to (153.6, 77.7)
- moved BOOT0 9.16 mm to (151.3, 75.1)
- moved CS1 9.00 mm to (150.9, 113.6), turned to 0 degrees
- moved C82 8.21 mm to (126.8, 84.7)
- moved C5 7.99 mm to (142.0, 90.7)
- moved R14 6.88 mm to (172.9, 93.8), turned to 90 degrees
- moved R15 6.63 mm to (130.5, 93.4)
- moved C11 6.28 mm to (124.2, 93.5)
- moved C1 5.71 mm to (142.0, 85.5)
- moved D2 5.11 mm to (129.0, 76.9), turned to 180 degrees
- moved J1 4.37 mm to (161.7, 87.5), turned to 180 degrees
- moved R56 4.28 mm to (157.6, 110.9)
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Routing:
- net +BATT: track 0.00 -> 92.4 mm, vias 0 -> 2
- net GND: track 0.00 -> 46.2 mm, vias 0 -> 30
- net +3.3V: track 0.00 -> 45.5 mm, vias 0 -> 2
- net /motorB/MB: track 0.00 -> 36.6 mm
- net /mcu/TIM3_CH2: track 0.00 -> 24.8 mm
- net /mcu/~{RESET}: track 0.00 -> 24.0 mm, vias 0 -> 2
- net Net-(U1-PB6): track 0.00 -> 21.5 mm
- net /motorA/MA: track 0.00 -> 20.5 mm
- net /mcu/IN_B2: track 0.00 -> 20.0 mm
- net /motorB/MA: track 0.00 -> 18.4 mm
- net Net-(J4-Pin_3): track 0.00 -> 17.1 mm
- net /mcu/TIM2_CH2: track 0.00 -> 15.8 mm
- net Net-(J2-Pin_3): track 0.00 -> 15.7 mm
- net Net-(J3-Pin_3): track 0.00 -> 15.0 mm
- net /mcu/TIM8_CH2: track 0.00 -> 13.8 mm
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- added copper zone on B.Cu, net GND
